File: buck.kicad_pcb (KiCad board)
At the start: 2 copper layers, 40.6 x 29.2 mm, 39 parts, among them U1 TPS5430

Commit message: Adjusted silk screen
Parts:
- moved REF*** 5.67 mm to (151.4, 113.3)
Changed lines of the file:
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@@
     (links 52)
     (no_connects 0)
-    (area 136.449999 88.824999 178.510001 118.185001)
+    (area 133.35 83.025 189.765558 121.920001)
     (thickness 1.6)
     (drawings 7)
@@
   )
   (module Symbols:KiCad-Logo2_6mm_SilkScreen (layer B.Cu)
-    (at 156.845 111.76 180)
+    (at 151.384 113.284 180)
     (descr "KiCad Logo")
     (tags "Logo KiCad")

Commit message: Fixed bottom silk
Other:
- board text added: "Buck Converter In: 8-36V Out: Adjustable (3A max) Bryan Orabutt"
- board text removed: "Buck Converter In: 8-36V Out: 5V/3A Bryan Orabutt"
Changed lines of the file:
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@@
     )
   )
-  (gr_text "Buck Converter\nIn: 8-36V\nOut: 5V/3A\n\nBryan Orabutt" (at 157.48 101.6) (layer B.SilkS)
-    (effects (font (size 1.5 1.5) (thickness 0.3)) (justify mirror))
+  (gr_text "Buck Converter\nIn: 8-36V\nOut: Adjustable (3A max)\n\nBryan Orabutt" (at 170.688 101.6) (layer B.SilkS)
+    (effects (font (size 1.5 1.5) (thickness 0.3)) (justify left mirror))
   )
   (dimension 29.21 (width 0.3) (layer Eco1.User)

Commit message: Added mounting holes
Parts:
- added REF**: MountingHole_2.2mm_M2, Mounting_Holes:MountingHole_2.2mm_M2, F.Cu at (178.6, 102.9)
- added REF**: MountingHole_2.2mm_M2, Mounting_Holes:MountingHole_2.2mm_M2, F.Cu at (136.7, 102.9)
- moved +5V- 3.35 mm to (138.4, 112.5)
- moved C1 3.18 mm to (154.9, 92.7)
- moved L1 1.27 mm to (146.1, 97.8)
Routing:
- net +5V: track 27.9 -> 29.8 mm
- net Net-(C1-Pad1): track 3.21 -> 4.08 mm
Other:
- board size 40.6 x 29.2 mm -> 47.8 x 29.2 mm
Changed lines of the file:
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@@
     (thickness 1.6)
     (drawings 7)
-    (tracks 28)
+    (tracks 27)
     (zones 0)
-    (modules 39)
+    (modules 41)
     (nets 14)
   )
@@
     (add_net GND)
   )
+  (module Mounting_Holes:MountingHole_2.2mm_M2 (layer F.Cu)
+    (at 178.562 102.87)
+    (descr "Mounting Hole 2.2mm, no annular, M2")
+    (tags "mounting hole 2.2mm no annular m2")
+    (attr virtual)
+    (fp_text reference REF** (at 0 -3.2) (layer F.SilkS) hide
+      (effects (font (size 1 1) (thickness 0.15)))
+    )
+    (fp_text value MountingHole_2.2mm_M2 (at 0 3.2) (layer F.Fab) hide
+      (effects (font (size 1 1) (thickness 0.15)))
+    )
+    (fp_text user %R (at 0.3 0) (layer F.Fab) hide
+      (effects (font (size 1 1) (thickness 0.15)))
+    )
+    (fp_circle (center 0 0) (end 2.2 0) (layer Cmts.User) (width 0.15))
+    (fp_circle (center 0 0) (end 2.45 0) (layer F.CrtYd) (width 0.05))
+    (pad 1 np_thru_hole circle (at 0 0) (size 2.2 2.2) (drill 2.2) (layers *.Cu *.Mask))
+  )
   (module footprints:SRR1208-220ML (layer F.Cu)
-    (at 144.78 97.79 270)
+    (at 146.05 97.79 270)
     (fp_text reference L1 (at 5.715 -7.62 270) (layer F.SilkS)
       (effects (font (size 1 1) (thickness 0.15)))
@@
   )
   (module Capacitors_SMD:C_0805_HandSoldering (layer F.Cu)
-    (at 153.035 95.25 90)
+    (at 154.94 92.71 90)
     (descr "Capacitor SMD 0805, hand soldering")
     (tags "capacitor 0805")
     (attr smd)
-    (fp_text reference C1 (at 3.155 0 180) (layer F.SilkS)
+    (fp_text reference C1 (at 0 -1.778 270) (layer F.SilkS)
       (effects (font (size 1 1) (thickness 0.15)))
     )
@@
     (tags "Diode 1206")
     (attr smd)
-    (fp_text reference +5V (at 0.278 1.905 180) (layer F.SilkS)
+    (fp_text reference +5V (at 4.596 0.127 180) (layer F.SilkS)
       (effects (font (size 1 1) (thickness 0.15)))
     )
@@
   )
   (module Terminal_Blocks:TerminalBlock_Pheonix_PT-3.5mm_2pol (layer F.Cu)
-    (at 141.605 111.45 90)
+    (at 138.43 112.522 90)
     (descr "2-way 3.5mm pitch terminal block, Phoenix PT series")
     (fp_text reference +5V- (at 1.75 5.715 90) (layer F.SilkS)
@@
     )
   )
+  (module Mounting_Holes:MountingHole_2.2mm_M2 (layer F.Cu)
+    (at 136.652 102.87)
+    (descr "Mounting Hole 2.2mm, no annular, M2")
+    (tags "mounting hole 2.2mm no annular m2")
+    (attr virtual)
+    (fp_text reference REF** (at 0 -3.2) (layer F.SilkS) hide
+      (effects (font (size 1 1) (thickness 0.15)))
+    )
+    (fp_text value MountingHole_2.2mm_M2 (at 0 3.2) (layer F.Fab) hide
+      (effects (font (size 1 1) (thickness 0.15)))
+    )
+    (fp_text user %R (at 0.3 0) (layer F.Fab) hide
+      (effects (font (size 1 1) (thickness 0.15)))
+    )
+    (fp_circle (center 0 0) (end 2.2 0) (layer Cmts.User) (width 0.15))
+    (fp_circle (center 0 0) (end 2.45 0) (layer F.CrtYd) (width 0.05))
+    (pad 1 np_thru_hole circle (at 0 0) (size 2.2 2.2) (drill 2.2) (layers *.Cu *.Mask))
+  )
   (gr_text "Buck Converter\nIn: 8-36V\nOut: Adjustable (3A max)\n\nBryan Orabutt" (at 170.688 101.6) (layer B.SilkS)
     (effects (font (size 1.5 1.5) (thickness 0.3)) (justify left mirror))
@@
     (arrow2b (pts (xy 182.879843 88.9) (xy 183.466264 90.026504)))
   )
-  (dimension 40.767 (width 0.3) (layer Eco1.User)
-    (gr_text "1.6050 in" (at 158.0515 84.375) (layer Eco1.User)
+  (dimension 47.752 (width 0.3) (layer Eco1.User)
+    (gr_text "1.8800 in" (at 157.734 84.502) (layer Eco1.User)
       (effects (font (size 1.5 1.5) (thickness 0.3)))
     )
-    (feature1 (pts (xy 178.435 88.9) (xy 178.435 83.025)))
-    (feature2 (pts (xy 137.668 88.9) (xy 137.668 83.025)))
-    (crossbar (pts (xy 137.668 85.725) (xy 178.435 85.725)))
-    (arrow1a (pts (xy 178.435 85.725) (xy 177.308496 86.311421)))
-    (arrow1b (pts (xy 178.435 85.725) (xy 177.308496 85.138579)))
-    (arrow2a (pts (xy 137.668 85.725) (xy 138.794504 86.311421)))
-    (arrow2b (pts (xy 137.668 85.725) (xy 138.794504 85.138579)))
-  )
-  (gr_line (start 178.435 118.11) (end 137.795 118.11) (layer Edge.Cuts) (width 0.15))
-  (gr_line (start 178.435 88.9) (end 178.435 118.11) (layer Edge.Cuts) (width 0.15))
-  (gr_line (start 137.795 88.9) (end 178.435 88.9) (layer Edge.Cuts) (width 0.15))
-  (gr_line (start 137.795 118.11) (end 137.795 88.9) (layer Edge.Cuts) (width 0.15))
-  (segment (start 155.97 97.155) (end 153.69 97.155) (width 0.1524) (layer F.Cu) (net 1))
-  (segment (start 153.69 97.155) (end 153.035 96.5) (width 0.1524) (layer F.Cu) (net 1))
+    (feature1 (pts (xy 181.61 88.9) (xy 181.61 83.152)))
+    (feature2 (pts (xy 133.858 88.9) (xy 133.858 83.152)))
+    (crossbar (pts (xy 133.858 85.852) (xy 181.61 85.852)))
+    (arrow1a (pts (xy 181.61 85.852) (xy 180.483496 86.438421)))
+    (arrow1b (pts (xy 181.61 85.852) (xy 180.483496 85.265579)))
+    (arrow2a (pts (xy 133.858 85.852) (xy 134.984504 86.438421)))
+    (arrow2b (pts (xy 133.858 85.852) (xy 134.984504 85.265579)))
+  )
+  (gr_line (start 181.61 118.11) (end 133.858 118.11) (layer Edge.Cuts) (width 0.15))
+  (gr_line (start 181.61 88.9) (end 181.61 118.11) (layer Edge.Cuts) (width 0.15))
+  (gr_line (start 133.858 88.9) (end 181.61 88.9) (layer Edge.Cuts) (width 0.15))
+  (gr_line (start 133.858 118.11) (end 133.858 88.9) (layer Edge.Cuts) (width 0.15))
+  (segment (start 155.97 97.155) (end 155.97 94.2126) (width 0.1524) (layer F.Cu) (net 1))
+  (segment (start 155.97 94.2126) (end 155.7174 93.96) (width 0.1524) (layer F.Cu) (net 1))
+  (segment (start 155.7174 93.96) (end 154.94 93.96) (width 0.1524) (layer F.Cu) (net 1))
   (segment (start 161.53 98.425) (end 163.0946 98.425) (width 0.6096) (layer F.Cu) (net 2))
   (segment (start 163.0946 98.425) (end 163.7296 97.79) (width 0.6096) (layer F.Cu) (net 2))
@@
   (segment (start 161.53 99.695) (end 159.4925 99.695) (width 0.6096) (layer F.Cu) (net 3))
   (segment (start 159.4925 99.695) (end 159.3525 99.835) (width 0.6096) (layer F.Cu) (net 3))
-  (segment (start 144.78 117.348) (end 141.605 114.173) (width 0.6096) (layer B.Cu) (net 4))
-  (segment (start 141.605 114.173) (end 141.605 111.45) (width 0.6096) (layer B.Cu) (net 4))
-  (segment (start 163.068 117.348) (end 144.78 117.348) (width 0.6096) (layer B.Cu) (net 4))
-  (segment (start 163.745001 116.670999) (end 163.068 117.348) (width 0.6096) (layer B.Cu) (net 4))
-  (segment (start 164.465 115.57) (end 163.745001 116.289999) (width 0.6096) (layer B.Cu) (net 4))
-  (segment (start 163.745001 116.289999) (end 163.745001 116.670999) (width 0.6096) (layer B.Cu) (net 4))
+  (segment (start 164.465 115.57) (end 162.687 117.348) (width 0.6096) (layer B.Cu) (net 4))
+  (segment (start 162.687 117.348) (end 141.4464 117.348) (width 0.6096) (layer B.Cu) (net 4))
+  (segment (start 141.4464 117.348) (end 138.43 114.3316) (width 0.6096) (layer B.Cu) (net 4))
+  (segment (start 138.43 114.3316) (end 138.43 112.522) (width 0.6096) (layer B.Cu) (net 4))
   (segment (start 173.83 92.71) (end 171.68 92.71) (width 0.1524) (layer F.Cu) (net 5))
   (segment (start 146.05 116.205) (end 143.51 116.205) (width 0.1524) (layer F.Cu) (net 6))
@@
     (polygon
       (pts
-        (xy 133.35 87.63) (xy 180.34 87.63) (xy 180.34 121.92) (xy 133.35 121.92)
+        (xy 133.35 87.63) (xy 182.88 87.63) (xy 182.88 123.19) (xy 133.35 121.92)
       )
     )
@@
       (pts
         (xy 173.355 120.65) (xy 173.355 98.425) (xy 163.195 98.425) (xy 163.195 95.885) (xy 166.37 95.885)
-        (xy 166.37 89.535) (xy 178.435 89.535) (xy 179.07 90.805) (xy 179.07 120.65)
+        (xy 166.37 87.63) (xy 177.8 87.63) (xy 185.42 87.63) (xy 185.42 121.285)
       )
     )
@@
       (pts
         (xy 160.655 97.79) (xy 162.56 97.79) (xy 162.56 95.25) (xy 165.735 95.25) (xy 165.735 90.805)
-        (xy 165.735 88.9) (xy 135.255 88.9) (xy 135.255 99.695) (xy 151.765 99.695) (xy 151.765 95.25)
-        (xy 156.21 95.25) (xy 156.21 90.805) (xy 161.29 90.805) (xy 161.29 94.615) (xy 160.655 94.615)
+        (xy 165.735 88.9) (xy 132.842 88.9) (xy 132.842 99.568) (xy 154.178 99.568) (xy 154.178 95.504)
+        (xy 156.21 95.504) (xy 156.21 90.805) (xy 161.29 90.805) (xy 161.29 94.615) (xy 160.655 94.615)
       )
     )
@@
     (polygon
       (pts
-        (xy 135.255 120.015) (xy 147.32 120.015) (xy 147.32 114.935) (xy 154.305 114.935) (xy 154.305 106.68)
-        (xy 158.115 106.68) (xy 158.115 104.775) (xy 154.305 104.775) (xy 154.305 100.33) (xy 135.255 100.33)
+        (xy 133.096 120.015) (xy 147.32 120.015) (xy 147.32 114.935) (xy 154.305 114.935) (xy 154.305 106.68)
+        (xy 158.115 106.68) (xy 158.115 104.775) (xy 154.305 104.775) (xy 154.305 100.33) (xy 133.096 100.33)
       )
     )

Commit message: Moved vias
Parts:
- moved REF** 0.51 mm to (158.1, 116.1)
- moved REF** 0.51 mm to (159.4, 114.8)
- moved REF** 0.51 mm to (159.4, 116.1)
- moved REF** 0.51 mm to (158.1, 114.8)
- moved REF** 0.51 mm to (159.4, 113.5)
- moved REF** 0.51 mm to (158.1, 113.5)
Changed lines of the file:
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@@
-(kicad_pcb (version 4) (host pcbnew 4.0.3-stable)
+(kicad_pcb (version 4) (host pcbnew 4.0.2+dfsg1-stable)
   (general
     (links 52)
     (no_connects 0)
-    (area 133.35 83.025 189.765558 121.920001)
+    (area 127.067457 83.002 189.915558 123.190001)
     (thickness 1.6)
     (drawings 7)
@@
   )
   (module footprints:via-0.7mm (layer F.Cu)
-    (at 158.115 115.57)
-    (fp_text reference REF** (at 0 1) (layer F.SilkS) hide
-      (effects (font (size 1 1) (thickness 0.15)))
-    )
-    (fp_text value via-0.7mm (at 0 -1) (layer F.Fab) hide
-      (effects (font (size 1 1) (thickness 0.15)))
-    )
-    (pad 1 thru_hole circle (at 0 0) (size 0.7 0.7) (drill 0.3302) (layers *.Cu)
-      (net 3 GND) (zone_connect 2))
-  )
-  (module footprints:via-0.7mm (layer F.Cu)
-    (at 158.115 114.3)
-    (fp_text reference REF** (at 0 1) (layer F.SilkS) hide
-      (effects (font (size 1 1) (thickness 0.15)))
-    )
-    (fp_text value via-0.7mm (at 0 -1) (layer F.Fab) hide
-      (effects (font (size 1 1) (thickness 0.15)))
-    )
-    (pad 1 thru_hole circle (at 0 0) (size 0.7 0.7) (drill 0.3302) (layers *.Cu)
-      (net 3 GND) (zone_connect 2))
-  )
-  (module footprints:via-0.7mm (layer F.Cu)
-    (at 158.115 113.03)
+    (at 158.115 116.078)
+    (fp_text reference REF** (at 0 1) (layer F.SilkS) hide
+      (effects (font (size 1 1) (thickness 0.15)))
+    )
+    (fp_text value via-0.7mm (at 0 -1) (layer F.Fab) hide
+      (effects (font (size 1 1) (thickness 0.15)))
+    )
+    (pad 1 thru_hole circle (at 0 0) (size 0.7 0.7) (drill 0.3302) (layers *.Cu)
+      (net 3 GND) (zone_connect 2))
+  )
+  (module footprints:via-0.7mm (layer F.Cu)
+    (at 158.115 114.808)
+    (fp_text reference REF** (at 0 1) (layer F.SilkS) hide
+      (effects (font (size 1 1) (thickness 0.15)))
+    )
+    (fp_text value via-0.7mm (at 0 -1) (layer F.Fab) hide
+      (effects (font (size 1 1) (thickness 0.15)))
+    )
+    (pad 1 thru_hole circle (at 0 0) (size 0.7 0.7) (drill 0.3302) (layers *.Cu)
+      (net 3 GND) (zone_connect 2))
+  )
+  (module footprints:via-0.7mm (layer F.Cu)
+    (at 158.115 113.538)
     (fp_text reference REF** (at 0 1) (layer F.SilkS) hide
       (effects (font (size 1 1) (thickness 0.15)))
@@
   )
   (module footprints:via-0.7mm (layer F.Cu)
-    (at 159.385 113.03)
-    (fp_text reference REF** (at 0 1) (layer F.SilkS) hide
-      (effects (font (size 1 1) (thickness 0.15)))
-    )
-    (fp_text value via-0.7mm (at 0 -1) (layer F.Fab) hide
-      (effects (font (size 1 1) (thickness 0.15)))
-    )
-    (pad 1 thru_hole circle (at 0 0) (size 0.7 0.7) (drill 0.3302) (layers *.Cu)
-      (net 3 GND) (zone_connect 2))
-  )
-  (module footprints:via-0.7mm (layer F.Cu)
-    (at 159.385 114.3)
-    (fp_text reference REF** (at 0 1) (layer F.SilkS) hide
-      (effects (font (size 1 1) (thickness 0.15)))
-    )
-    (fp_text value via-0.7mm (at 0 -1) (layer F.Fab) hide
-      (effects (font (size 1 1) (thickness 0.15)))
-    )
-    (pad 1 thru_hole circle (at 0 0) (size 0.7 0.7) (drill 0.3302) (layers *.Cu)
-      (net 3 GND) (zone_connect 2))
-  )
-  (module footprints:via-0.7mm (layer F.Cu)
-    (at 159.385 115.57)
-    (fp_text reference REF** (at 0 1) (layer F.SilkS) hide
-      (effects (font (size 1 1) (thickness 0.15)))
+    (at 159.385 113.538)
+    (fp_text reference REF** (at 0 1) (layer F.SilkS) hide
+      (effects (font (size 1 1) (thickness 0.15)))
+    )
+    (fp_text value via-0.7mm (at 0 -1) (layer F.Fab) hide
+      (effects (font (size 1 1) (thickness 0.15)))
+    )
+    (pad 1 thru_hole circle (at 0 0) (size 0.7 0.7) (drill 0.3302) (layers *.Cu)
+      (net 3 GND) (zone_connect 2))
+  )
+  (module footprints:via-0.7mm (layer F.Cu)
+    (at 159.385 114.808)
+    (fp_text reference REF** (at 0 1) (layer F.SilkS) hide
+      (effects (font (size 1 1) (thickness 0.15)))
+    )
+    (fp_text value via-0.7mm (at 0 -1) (layer F.Fab) hide
+      (effects (font (size 1 1) (thickness 0.15)))
+    )
+    (pad 1 thru_hole circle (at 0 0) (size 0.7 0.7) (drill 0.3302) (layers *.Cu)
+      (net 3 GND) (zone_connect 2))
+  )
+  (module footprints:via-0.7mm (layer F.Cu)
+    (at 159.385 116.078)
+    (fp_text reference REF** (at 0 1) (layer F.SilkS) hide
+      (effects (font (size 1 1) (thickness 0.15)))
